File: hdmi.kicad_sch (KiCad schematic)
At the start: 1 part

Commit message: HW Rev 2.0
Parts:
- HDMI1: footprint LIBS:HDMI -> Connector_Video:HDMI_A_Contact_Technology_HDMI-19APL2_Horizontal
Changed lines of the file:
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@@
 	(generator "eeschema")
 	(generator_version "8.0")
-	(paper "A4")
+	(paper "A3")
 	(title_block
 		(title "HDMI to VGA Passive Adapter")
-		(date "2024-12-01")
-		(rev "1.0")
+		(date "2024-12-29")
+		(rev "2.0")
 		(company "Mikhail Matveev")
 	)
@@
 			)
 		)
-		(property "Footprint" "LIBS:HDMI"
+		(property "Footprint" "Connector_Video:HDMI_A_Contact_Technology_HDMI-19APL2_Horizontal"
 			(at 50.8 88.9 0)
 			(effects
