File: softcomp.kicad_sch (KiCad schematic)
At the start: 10 parts

Commit message: HW Rev 2.0
Parts:
- added H1, H2, H3, H4: MountingHole, MountingHole:MountingHole_2.1mm, symbol Mechanical:MountingHole
Other:
- title: Frank -> HDMI to VGA Passive Adapter
