File: hdmi2vgaP.kicad_pcb (KiCad board)
At the start: 2 copper layers, 54.4 x 26.4 mm, 27 parts, among them J1 HDMI, J2 VGA, J3 Composite

Commit message: Updates to HW Rev 1.0
Other:
- board text added: "HDMI>VGA"
- board text added: "HW Rev 1.0"
- board text added: "rh1.dev"
Changed lines of the file:
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@@
 		(layer "Edge.Cuts")
+	)
+	(gr_text "HW Rev 1.0"
+		(at 97 66.6 0)
+		(layer "B.Cu")
+		(effects
+			(font
+				(size 1 1)
+				(thickness 0.15)
+			)
+			(justify right bottom mirror)
+		)
+	)
+	(gr_text "HW Rev 1.0"
+		(at 97 66.6 0)
+		(layer "B.SilkS")
+		(effects
+			(font
+				(size 1 1)
+				(thickness 0.15)
+			)
+			(justify right bottom mirror)
+		)
+	)
+	(gr_text "HDMI>VGA"
+		(at 83.6 58 0)
+		(layer "B.SilkS")
+		(effects
+			(font
+				(face "PT Sans Caption")
+				(size 3 3)
+				(thickness 0.15)
+			)
+			(justify left bottom mirror)
+		)
+		(render_cache "HDMI>VGA" 0
+			(polygon
+				(pts
+					(xy 81.304361 56.17695) (xy 82.802058 56.17695) (xy 82.802058 57.49) (xy 83.22411 57.49) (xy 83.22411 54.535638)
+					(xy 82.802058 54.535638) (xy 82.802058 55.801793) (xy 81.304361 55.801793) (xy 81.304361 54.535638)
+					(xy 80.882309 54.535638) (xy 80.882309 57.49) (xy 81.304361 57.49)
+				)
+			)
+			(polygon
+				(pts
+					(xy 79.331538 54.488958) (xy 79.482065 54.490942) (xy 79.569615 54.492899) (xy 79.718736 54.497536)
+					(xy 79.800399 54.500401) (xy 79.951011 54.507794) (xy 79.998441 54.51096) (xy 80.14665 54.526845)
+					(xy 80.14665 57.498792) (xy 80.140639 57.499794) (xy 79.992777 57.513447) (xy 79.909315 57.517981)
+					(xy 79.758304 57.523705) (xy 79.66416 57.527002) (xy 79.511374 57.532498) (xy 79.468012 57.533992)
+					(xy 79.319399 57.536894) (xy 79.215833 57.534845) (xy 79.067782 57.524086) (xy 78.906125 57.499878)
+					(xy 78.756389 57.463118) (xy 78.59986 57.405736) (xy 78.474863 57.344001) (xy 78.344632 57.263573)
+					(xy 78.227865 57.172611) (xy 78.112595 57.05769) (xy 78.055813 56.988639) (xy 77.966316 56.856773)
+					(xy 77.893164 56.715171) (xy 77.836357 56.563831) (xy 77.806973 56.459022) (xy 77.774297 56.299297)
+					(xy 77.755299 56.136558) (xy 77.749895 55.989371) (xy 78.196859 55.989371) (xy 78.202011 56.128075)
+					(xy 78.21958 56.277342) (xy 78.249616 56.423147) (xy 78.280757 56.525179) (xy 78.345328 56.667924)
+					(xy 78.431332 56.798304) (xy 78.519775 56.894975) (xy 78.636236 56.986603) (xy 78.772784 57.062819)
+					(xy 78.841939 57.091316) (xy 78.995382 57.13382) (xy 79.150734 57.155555) (xy 79.302547 57.161737)
+					(xy 79.387543 57.159539) (xy 79.513572 57.155143) (xy 79.642533 57.151479) (xy 79.724598 57.144884)
+					(xy 79.724598 54.88515) (xy 79.640334 54.87709) (xy 79.517969 54.868297) (xy 79.383147 54.8639)
+					(xy 79.256385 54.8639) (xy 79.199479 54.864834) (xy 79.039966 54.878841) (xy 78.882444 54.914118)
+					(xy 78.745673 54.970146) (xy 78.649228 55.026475) (xy 78.52345 55.124363) (xy 78.420341 55.238325)
+					(xy 78.363647 55.321947) (xy 78.295434 55.455968) (xy 78.247418 55.600293) (xy 78.227718 55.686781)
+					(xy 78.205203 55.833252) (xy 78.196859 55.989371) (xy 77.749895 55.989371) (xy 77.755711 55.829499)
+					(xy 77.773159 55.675947) (xy 77.802239 55.528714) (xy 77.842951 55.387801) (xy 77.874146 55.303566)
+					(xy 77.942107 55.16132) (xy 78.025254 55.031129) (xy 78.123586 54.912993) (xy 78.197354 54.84132)
+					(xy 78.320854 54.745306) (xy 78.459771 54.663087) (xy 78.596196 54.601584) (xy 78.650417 54.581418)
+					(xy 78.803946 54.53734) (xy 78.948954 54.510342) (xy 79.103918 54.494143) (xy 79.268841 54.488743)
+				)
+			)
+			(polygon
+				(pts
+					(xy 74.655582 55.586371) (xy 74.60942 55.113761) (xy 74.626273 55.113761) (xy 74.807257 55.523356)
+					(xy 75.630844 56.833475) (xy 75.756873 56.833475) (xy 76.622226 55.519692) (xy 76.79515 55.118157)
+					(xy 76.816399 55.118157) (xy 76.748988 55.582707) (xy 76.748988 57.49) (xy 77.145394 57.49) (xy 77.145394 54.535638)
+					(xy 76.828855 54.535638) (xy 75.828681 56.044326) (xy 75.672609 56.365261) (xy 75.663817 56.365261)
+					(xy 75.516538 56.035533) (xy 74.566922 54.535638) (xy 74.233531 54.535638) (xy 74.233531 57.49)
+					(xy 74.655582 57.49)
+				)
+			)
+			(polygon
+				(pts
+					(xy 73.249476 54.817006) (xy 73.587264 54.817006) (xy 73.587264 54.535638) (xy 72.489637 54.535638)
+					(xy 72.489637 54.817006) (xy 72.827424 54.817006) (xy 72.827424 57.208632) (xy 72.489637 57.208632)
+					(xy 72.489637 57.49) (xy 73.587264 57.49) (xy 73.587264 57.208632) (xy 73.249476 57.208632)
+				)
+			)
+			(polygon
+				(pts
+					(xy 70.05478 56.00769) (xy 70.05478 56.168157) (xy 71.827983 57.161737) (xy 72.000907 56.857655)
+					(xy 70.920132 56.248757) (xy 70.49808 56.091953) (xy 70.915736 55.956399) (xy 72.022156 55.351165)
+					(xy 71.853628 55.051479)
+				)
+			)
+			(polygon
+				(pts
+					(xy 68.631088 56.505945) (xy 68.521179 56.966831) (xy 68.512386 56.966831) (xy 68.398813 56.497152)
+					(xy 67.638974 54.535638) (xy 67.216922 54.535638) (xy 68.441311 57.536894) (xy 68.652337 57.536894)
+					(xy 69.892847 54.535638) (xy 69.42903 54.535638)
+				)
+			)
+			(polygon
+				(pts
+					(xy 65.885554 55.989371) (xy 64.779134 55.989371) (xy 64.779134 57.295826) (xy 64.903818 57.373573)
+					(xy 64.960851 57.399874) (xy 65.105648 57.451581) (xy 65.186531 57.473879) (xy 65.331555 57.504293)
+					(xy 65.433461 57.520041) (xy 65.582441 57.534113) (xy 65.682588 57.536894) (xy 65.831836 57.531261)
+					(xy 65.993061 57.511458) (xy 66.147216 57.477397) (xy 66.246057 57.446769) (xy 66.386629 57.388248)
+					(xy 66.516537 57.314079) (xy 66.63578 57.22426) (xy 66.697418 57.167599) (xy 66.798912 57.053495)
+					(xy 66.887423 56.923858) (xy 66.962951 56.778688) (xy 66.999302 56.691325) (xy 67.047387 56.540933)
+					(xy 67.081734 56.377718) (xy 67.100517 56.224386) (xy 67.108782 56.061236) (xy 67.109211 56.012819)
+					(xy 67.104548 55.864192) (xy 67.087323 55.701278) (xy 67.057405 55.549654) (xy 67.014794 55.40932)
+					(xy 66.976587 55.315994) (xy 66.905054 55.177508) (xy 66.823813 55.052212) (xy 66.720812 54.927018)
+					(xy 66.632205 54.841186) (xy 66.509677 54.74532) (xy 66.379499 54.665451) (xy 66.24167 54.601579)
+					(xy 66.161793 54.573007) (xy 66.016004 54.532274) (xy 65.870447 54.504872) (xy 65.70899 54.49006)
+					(xy 65.644487 54.488743) (xy 65.495401 54.491294) (xy 65.347424 54.500109) (xy 65.19441 54.519)
+					(xy 65.182868 54.520983) (xy 65.033723 54.551357) (xy 64.892123 54.59294) (xy 64.876587 54.598653)
+					(xy 64.977704 54.95769) (xy 65.133981 54.90823) (xy 65.286205 54.881852) (xy 65.439237 54.868388)
+					(xy 65.610781 54.8639) (xy 65.764733 54.873575) (xy 65.918201 54.902598) (xy 65.988869 54.922519)
+					(xy 66.135109 54.982844) (xy 66.259152 55.061068) (xy 66.326657 55.116692) (xy 66.43083 55.230207)
+					(xy 66.512383 55.355083) (xy 66.56919 55.472065) (xy 66.617876 55.619012) (xy 66.646277 55.768394)
+					(xy 66.65926 55.914802) (xy 66.661514 56.012819) (xy 66.65537 56.173484) (xy 66.636939 56.321629)
+					(xy 66.602048 56.471553) (xy 66.583845 56.527194) (xy 66.522757 56.667473) (xy 66.439724 56.80036)
+					(xy 66.366224 56.886231) (xy 66.254701 56.98223) (xy 66.117837 57.062276) (xy 66.037229 57.095059)
+					(xy 65.88971 57.135691) (xy 65.732918 57.15757) (xy 65.623237 57.161737) (xy 65.469862 57.153159)
+					(xy 65.355059 57.134626) (xy 65.213284 57.094166) (xy 65.129378 57.056957) (xy 65.129378 56.317634)
+					(xy 65.885554 56.239965)
+				)
+			)
+			(polygon
+				(pts
+					(xy 64.515352 57.49) (xy 64.10136 57.49) (xy 63.789218 56.692791) (xy 62.620516 56.692791) (xy 62.299581 57.49)
+					(xy 61.860676 57.49) (xy 62.318174 56.364528) (xy 62.742882 56.364528) (xy 63.662456 56.364528)
+					(xy 63.320272 55.529218) (xy 63.206699 55.066866) (xy 63.197906 55.066866) (xy 63.084333 55.520425)
+					(xy 62.742882 56.364528) (xy 62.318174 56.364528) (xy 63.080669 54.488743) (xy 63.299755 54.488743)
+				)
+			)
+		)
+	)
+	(gr_text "rh1.dev"
+		(at 97.2 69 0)
+		(layer "B.SilkS")
+		(effects
+			(font
+				(size 0.8 0.8)
+				(thickness 0.13)
+			)
+			(justify right bottom mirror)
+		)
+	)
+	(dimension
+		(type aligned)
+		(layer "Dwgs.User")
+		(pts
+			(xy 55.8 57.2) (xy 110.189999 57.198485)
+		)
+		(height -27.20584)
+		(gr_text "54.3900 mm"
+			(at 82.99421 28.843402 0.001596992126)
+			(layer "Dwgs.User")
+			(effects
+				(font
+					(size 1 1)
+					(thickness 0.15)
+				)
+			)
+		)
+		(format
+			(prefix "")
+			(suffix "")
+			(units 3)
+			(units_format 1)
+			(precision 4)
+		)
+		(style
+			(thickness 0.1)
+			(arrow_length 1.27)
+			(text_position_mode 0)
+			(extension_height 0.58642)
+			(extension_offset 0.5) keep_text_aligned)
+	)
+	(dimension
+		(type aligned)
+		(layer "Dwgs.User")
+		(pts
+			(xy 93.2 44) (xy 93.2 70.4)
+		)
+		(height -29.2)
+		(gr_text "26.4000 mm"
+			(at 121.25 57.2 90)
+			(layer "Dwgs.User")
+			(effects
+				(font
+					(size 1 1)
+					(thickness 0.15)
+				)
+			)
+		)
+		(format
+			(prefix "")
+			(suffix "")
+			(units 3)
+			(units_format 1)
+			(precision 4)
+		)
+		(style
+			(thickness 0.1)
+			(arrow_length 1.27)
+			(text_position_mode 0)
+			(extension_height 0.58642)
+			(extension_offset 0.5) keep_text_aligned)
 	)
 	(segment

Commit message: HW Rev 2.0
Parts:
- removed REF** (x4): MountingHole_2.1mm, LIBS:MountingHole_2.1mm
- added H1: MountingHole, MountingHole:MountingHole_2.1mm, F.Cu at (92.6, 23.2)
- added H2: MountingHole, MountingHole:MountingHole_2.1mm, F.Cu at (92.6, 49.8)
- added H3: MountingHole, MountingHole:MountingHole_2.1mm, F.Cu at (68.4, 49.8)
- added H4: MountingHole, MountingHole:MountingHole_2.1mm, F.Cu at (68.4, 23.2)
- HDMI1: footprint LIBS:HDMI -> Connector_Video:HDMI_A_Contact_Technology_HDMI-19APL2_Horizontal
- moved J3 35.5 mm to (68.6, 42.5), turned to 180 degrees
- moved VGA1 31.9 mm to (97.2, 32.2), turned to 90 degrees
- moved J1 31.8 mm to (71.2, 42.5), turned to 180 degrees
- moved C1 31.1 mm to (75.6, 49.1), turned to 90 degrees
- moved SC1 28.2 mm to (83.6, 26.3)
- moved J2 28.0 mm to (73.9, 42.5), turned to 180 degrees
- moved HDMI1 27.4 mm to (61.2, 36.2), turned to -90 degrees
- moved R10 26.9 mm to (91.6, 42.0), turned to 0 degrees
- moved R9 26.5 mm to (91.6, 38.0), turned to 180 degrees
- moved R8 25.9 mm to (91.6, 40.0), turned to 0 degrees
- moved R6 24.8 mm to (82.4, 46.0), turned to 180 degrees
- moved R7 23.9 mm to (86.6, 50.2), turned to 0 degrees
- moved R5 22.9 mm to (82.4, 44.0), turned to 180 degrees
- moved R15 22.5 mm to (82.4, 34.0), turned to 0 degrees
- moved R12 22.4 mm to (91.6, 34.0), turned to 180 degrees
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Routing:
- net /HDMI/D2P: track 23.8 -> 55.5 mm
- net /HDMI/D2N: track 78.0 -> 48.9 mm, vias 1 -> 2
- net /Soft Composite/D0P: track 28.9 -> 55.4 mm
- net /HDMI/CLKN: track 38.4 -> 12.3 mm
- net /HDMI/CLKP: track 37.5 -> 11.6 mm
- net /HDMI/D0N: track 33.8 -> 10.7 mm
- net /VGA/VGA_RH: track 13.3 -> 33.8 mm, vias 0 -> 1
- net /Soft Composite/CVBS: track 14.7 -> 34.0 mm
- net /Soft Composite/D0N: track 27.4 -> 45.9 mm
- net /HDMI/D0P: track 28.2 -> 10.9 mm
- net /HDMI/VBUS: track 45.1 -> 29.9 mm, vias 2 -> 1
- net /VGA/VGA_BH: track 7.47 -> 22.5 mm, vias 0 -> 1
- net /VGA/VGA_GH: track 9.17 -> 22.1 mm, vias 0 -> 1
- net Net-(L1-A): track 16.9 -> 5.55 mm
- net Net-(C1-Pad1): track 9.14 -> 20.4 mm
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Other:
- board size 54.4 x 26.4 mm -> 44.7 x 31.4 mm
- board text added: "HW REV 2.0"
- board text added: "RH1.DEV"
- board text removed: "HW Rev 1.0"
- board text removed: "rh1.dev"

Commit message: Minor updates
Parts:
- R7: value 10K -> 1K
Changed lines of the file:
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@@
 	(title_block
 		(title "HDMI to VGA Passive Adapter")
-		(date "2024-12-29")
+		(date "2025-01-14")
 		(rev "2.0")
 		(company "Mikhail Matveev")
@@
 			)
 		)
-		(property "Value" "10K"
+		(property "Value" "1K"
 			(at 0 1.65 0)
 			(layer "F.Fab")
