File: hdmi2vgaP.kicad_sch (KiCad schematic)
At the start: 11 parts, among them J1 HDMI, J2 VGA, J3 Composite

Commit message: Minor updates
Parts:
- R7: value 10K -> 1K
Changed lines of the file:
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@@
 	(title_block
 		(title "HDMI to VGA Passive Adapter")
-		(date "2024-12-29")
+		(date "2025-01-14")
 		(rev "2.0")
 		(company "Mikhail Matveev")
@@
 			)
 		)
-		(property "Value" "10K"
+		(property "Value" "1K"
 			(at 57.404 88.9 90)
 			(effects
